File: hw_design/bxdrone.sch (EAGLE design)
At the start: 23 parts, among them J1 POWER_JACKPTH_BREAD

Commit message: Modifications on schematic
Connections:
- net RX: now also J8.2; no longer J7.1
- net TX: now also J7.1; no longer J8.2
Changed lines of the file:
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@@
 </segment>
 <segment>
-<wire x1="226.06" y1="25.4" x2="208.28" y2="25.4" width="0.1524" layer="91"/>
-<label x="208.28" y="25.4" size="1.778" layer="95"/>
-<pinref part="J7" gate="G$1" pin="1"/>
+<wire x1="226.06" y1="48.26" x2="208.28" y2="48.26" width="0.1524" layer="91"/>
+<label x="208.28" y="48.26" size="1.778" layer="95"/>
+<pinref part="J8" gate="G$1" pin="2"/>
 </segment>
 </net>
@@
 </segment>
 <segment>
-<wire x1="226.06" y1="48.26" x2="208.28" y2="48.26" width="0.1524" layer="91"/>
-<label x="208.28" y="48.26" size="1.778" layer="95"/>
-<pinref part="J8" gate="G$1" pin="2"/>
+<wire x1="226.06" y1="25.4" x2="208.28" y2="25.4" width="0.1524" layer="91"/>
+<label x="208.28" y="25.4" size="1.778" layer="95"/>
+<pinref part="J7" gate="G$1" pin="1"/>
 </segment>
 </net>
